Commit message: update

File: urdf/amr_mtt.xacro (robot description, xacro)
@@ -2,21 +2,21 @@
 <robot xmlns:xacro="http://www.ros.org/wiki/xacro" name="amr_mtt">
     <!--................................ XACRO CONSTANTS .............................. -->
-    <xacro:property name="chassis_mass" value="70"/>
+    <xacro:property name="chassis_mass" value="60"/>
     <xacro:property name="chassis_length" value="0.9"/>
     <xacro:property name="chassis_width" value="0.64"/>
-    <xacro:property name="chassis_height" value="0.19"/>
+    <xacro:property name="chassis_height" value="0.2"/>
     <xacro:property name="traction_wheel_mass" value="1"/>
     <xacro:property name="traction_wheel_base" value="0.88"/>
-    <xacro:property name="traction_max_wheel_torque" value="20000"/>
-    <xacro:property name="traction_wheel_friction" value="5.0"/>
+    <xacro:property name="traction_max_wheel_torque" value="150000"/>
+    <xacro:property name="traction_wheel_friction" value="3.0"/>
     <xacro:property name="trolley_wheel_mass" value="0.1"/>
-    <xacro:property name="trolley_track_width" value="0.54"/>
+    <xacro:property name="trolley_track_width" value="0.5"/>
     <xacro:property name="trolley_wheel_friction" value="0.0"/>
     <xacro:property name="trolley_wheel_radius" value="0.06"/>
     <!-- a small constant -->
     <xacro:property name="eps" value="0.002"/>
-    <xacro:property name="traction_wheel_radius" value="0.1"/>
+    <xacro:property name="traction_wheel_radius" value="0.08"/>
     <xacro:property name="traction_wheel_width" value="0.05"/>
-    <xacro:property name="traction_track_width" value="0.6"/>
+    <xacro:property name="traction_track_width" value="0.436"/>
     <xacro:property name="two_d_lidar_update_rate" value="30"/>
     <xacro:property name="two_d_lidar_sample_size" value="361"/>
@@ -89,38 +89,82 @@
     </joint>
     <!-- ................................ WHEELS ..................................... -->
-    <xacro:trolley_wheel cardinality="front" dexterity="left" origin_x="${chassis_length/2}" origin_y="${trolley_track_width/2}" origin_z="-${trolley_wheel_radius+chassis_height/2}"/>
-    <xacro:trolley_wheel cardinality="front" dexterity="right" origin_x="${chassis_length/2}" origin_y="-${trolley_track_width/2}" origin_z="-${trolley_wheel_radius+chassis_height/2}"/>
-    <xacro:trolley_wheel cardinality="back" dexterity="left" origin_x="-${chassis_length/2}" origin_y="${trolley_track_width/2}" origin_z="-${trolley_wheel_radius+chassis_height/2}"/>
-    <xacro:trolley_wheel cardinality="back" dexterity="right" origin_x="-${chassis_length/2}" origin_y="-${trolley_track_width/2}" origin_z="-${trolley_wheel_radius+chassis_height/2}"/>
+    <xacro:trolley_wheel cardinality="front" dexterity="left" origin_x="${chassis_length/2-0.10}" origin_y="${trolley_track_width/2}" origin_z="-${trolley_wheel_radius+chassis_height/2}"/>
+    <xacro:trolley_wheel cardinality="front" dexterity="right" origin_x="${chassis_length/2-0.10}" origin_y="-${trolley_track_width/2}" origin_z="-${trolley_wheel_radius+chassis_height/2}"/>
+    <xacro:trolley_wheel cardinality="back" dexterity="left" origin_x="-${chassis_length/2-0.10}" origin_y="${trolley_track_width/2}" origin_z="-${trolley_wheel_radius+chassis_height/2}"/>
+    <xacro:trolley_wheel cardinality="back" dexterity="right" origin_x="-${chassis_length/2-0.10}" origin_y="-${trolley_track_width/2}" origin_z="-${trolley_wheel_radius+chassis_height/2}"/>
     <xacro:traction_wheel cardinality="middle" dexterity="left" origin_x="0" origin_y="${traction_track_width/2}" origin_z="-${chassis_height/2+2*trolley_wheel_radius+eps-traction_wheel_radius}"/>
     <xacro:traction_wheel cardinality="middle" dexterity="right" origin_x="0" origin_y="-${traction_track_width/2}" origin_z="-${chassis_height/2+2*trolley_wheel_radius+eps-traction_wheel_radius}"/>
     <!-- ............................. 2D LIDAR ........................................ -->
+    <!-- ========================================================= -->
+    <!-- .......................... FRONT LIDAR .................... -->
+    <!-- ========================================================= -->
     <xacro:if value="$(arg two_d_lidar_enabled)">
-        <link name="two_d_lidar">
-            <collision>
-                <origin xyz="0 0 0" rpy="0 0 0" />
-                <geometry>
-                    <cylinder length="0.06" radius="0.075"/>
-                </geometry>
-            </collision>
-            <visual>
-                <origin xyz="0 0 0" rpy="0 0 0" />
-                <geometry>
-                    <cylinder length="0.06" radius="0.075"/>
-                </geometry>
-                <material name="aluminium"/>
-            </visual>
-            <inertial>
-                <origin xyz="0 0 0" rpy="0 0 0" />
+        <link name="L_F_Lidar_Link">
+            <collision>
+                <origin xyz="0 0 0" rpy="0 0 0"/>
+                <geometry>
+                    <!-- <mesh filename="package://amr_mtt/meshes/amr_mtt_model/L_F_Lidar_Link.STL" scale="1 1 1"/> -->
+                    <mesh filename="file://$(find amr_mtt)/meshes/amr_mtt_model/L_F_Lidar_Link.STL" scale="1 1 1"/>
+                </geometry>
+            </collision>
+            <visual>
+                <origin xyz="0 0 0" rpy="0 0 0"/>
+                <geometry>
+                    <!-- <mesh filename="package://amr_mtt/meshes/amr_mtt_model/L_F_Lidar_Link.STL" scale="1 1 1"/> -->
+                    <mesh filename="file://$(find amr_mtt)/meshes/amr_mtt_model/L_F_Lidar_Link.STL" scale="1 1 1"/>
+                </geometry>
+                <material name="blue">
+                    <color rgba="0 0 1 1" />
+                </material>
+            </visual>
+            <inertial>
+                <origin xyz="0 0 0" rpy="0 0 0"/>
                 <mass value="0.1"/>
                 <xacro:cylinder_inertia m="0.1" r="0.075" h="0.06"/>
             </inertial>
         </link>
-        <joint name="two_d_lidar_joint" type="fixed">
-            <parent link="base_link"/>
-            <child link="two_d_lidar"/>
-            <origin xyz="0.0 0 0.08" rpy="0 0 0" />
-        </joint>
-        <gazebo reference="two_d_lidar">
+        <joint name="L_F_Lidar_joint" type="fixed">
+            <parent link="base_link"/>
+            <child link="L_F_Lidar_Link"/>
+            <origin xyz="0.33905 0.18905 0.18259" rpy="3.1416 0 0.7854"/>
+        </joint>
+        <gazebo reference="L_F_Lidar_Link">
+            <material>Gazebo/White</material>
+        </gazebo>
+    </xacro:if>
+    <!-- ========================================================= -->
+    <!-- .......................... REAR LIDAR .................... -->
+    <!-- ========================================================= -->
+    <xacro:if value="$(arg two_d_lidar_enabled)">
+        <link name="R_B_Lidar_Link">
+            <collision>
+                <origin xyz="0 0 0" rpy="0 0 0"/>
+                <geometry>
+                    <!-- <mesh filename="package://amr_mtt/meshes/amr_mtt_model/R_B_Lidar_Link.STL" scale="1 1 1"/> -->
+                    <mesh filename="file://$(find amr_mtt)/meshes/amr_mtt_model/R_B_Lidar_Link.STL" scale="1 1 1"/>
+                </geometry>
+            </collision>
+            <visual>
+                <origin xyz="0 0 0" rpy="0 0 0"/>
+                <geometry>
+                    <mesh filename="file://$(find amr_mtt)/meshes/amr_mtt_model/R_B_Lidar_Link.STL" scale="1 1 1"/>
+                </geometry>
+                <material name="blue">
+                    <color rgba="0 0 1 1" />
+                </material>
+            </visual>
+            <inertial>
+                <origin xyz="0 0 0" rpy="0 0 0"/>
+                <mass value="0.1"/>
+                <xacro:cylinder_inertia m="0.1" r="0.075" h="0.06"/>
+            </inertial>
+        </link>
+        <joint name="R_B_Lidar_joint" type="fixed">
+            <parent link="base_link"/>
+            <child link="R_B_Lidar_Link"/>
+            <!-- จุดติดตั้งด้านหลัง -->
+            <origin xyz="-0.33905 -0.18905 0.18259" rpy="-3.1416 0 -0.7854"/>
+        </joint>
+        <gazebo reference="R_B_Lidar_Link">
             <material>Gazebo/White</material>
         </gazebo>
@@ -140,13 +184,16 @@
                 <origin xyz="0 0 0" rpy="0 0 0" />
                 <geometry>
-                    <box size="0.07 0.3 0.09"/>
-                </geometry>
-            </collision>
-            <visual>
-                <origin xyz="0 0 0" rpy="0 0 0" />
-                <geometry>
-                    <mesh filename="file://$(find amr_mtt)/meshes/kinect/d415.dae"/>
-                </geometry>
-                <material name="black"/>
+                    <mesh filename="file://$(find amr_mtt)/meshes/amr_mtt_model/F_Cam_Link.STL" scale="1 1 1"/>
+                </geometry>
+            </collision>
+            <visual>
+                <origin xyz="0 0 0" rpy="0 0 0" />
+                <geometry>
+                    <!-- <mesh filename="file://$(find amr_mtt)/meshes/kinect/d415.dae"/> -->
+                    <mesh filename="file://$(find amr_mtt)/meshes/amr_mtt_model/F_Cam_Link.STL" scale="1 1 1"/>
+                </geometry>
+                <material name="red">
+                    <color rgba="1 0 0 1" />
+                </material>
             </visual>
             <inertial>
@@ -156,5 +203,5 @@
         </link>
         <joint name="kinect_camera_joint" type="fixed">
-            <origin rpy="0 0 0" xyz="${chassis_length/2} 0 ${chassis_height/7}"/>
+            <origin rpy="0 0 0" xyz="${chassis_length/2} 0 0.26"/>
             <parent link="base_link"/>
             <child link="kinect_camera"/>
@@ -174,13 +221,15 @@
                 <origin xyz="0 0 0" rpy="0 0 0" />
                 <geometry>
-                    <box size="0.07 0.3 0.09"/>
-                </geometry>
-            </collision>
-            <visual>
-                <origin xyz="0 0 0" rpy="0 0 0" />
-                <geometry>
-                    <mesh filename="file://$(find amr_mtt)/meshes/kinect/d415.dae"/>
-                </geometry>
-                <material name="black"/>
+                    <mesh filename="file://$(find amr_mtt)/meshes/amr_mtt_model/F_Cam_Link.STL" scale="1 1 1"/>
+                </geometry>
+            </collision>
+            <visual>
+                <origin xyz="0 0 0" rpy="0 0 0" />
+                <geometry>
+                    <mesh filename="file://$(find amr_mtt)/meshes/amr_mtt_model/F_Cam_Link.STL" scale="1 1 1"/>
+                </geometry>
+                <material name="red">
+                    <color rgba="1 0 0 1" />
+                </material>
             </visual>
             <inertial>
@@ -190,5 +239,5 @@
         </link>
         <joint name="stereo_camera_joint" type="fixed">
-            <origin rpy="0 0 0" xyz="${chassis_length/2} 0 ${chassis_height/7}"/>
+            <origin rpy="0 0 0" xyz="${chassis_length/2} 0 0.26"/>
             <parent link="base_link"/>
             <child link="stereo_camera"/>
@@ -201,48 +250,3 @@
         </joint>
     </xacro:if>
-    <!-- ............................. ROOF ........................................ -->
-    <link name="roof_link">
-        <collision>
-            <origin xyz="0 0 0" rpy="0 0 0" />
-            <geometry>
-                <box size="${chassis_length} ${chassis_width} 0.015"/>
-            </geometry>
-        </collision>
-        <inertial>
-            <mass value="1"/>
-            <xacro:box_inertia m="1" x="1" y="0.6" z = "0.015"/>
-        </inertial>
-    </link>
-    <joint name="roof joint" type="fixed">
-        <parent link="chassis_link"/>
-        <child link="roof_link"/>
-        <origin xyz="0 0 0.16" rpy="0 0 0" />
-    </joint>
-    <!-- ............................. CONVEYOR ........................................ -->
-    <xacro:if value="$(arg conveyor_enabled)">
-        <link name="conveyor_belt">
-            <collision>
-                <origin xyz="0 0 0" rpy="0 0 0" />
-                <geometry>
-                    <box size="1 0.6 0.015"/>
-                </geometry>
-            </collision>
-            <visual>
-                <origin xyz="0 0 0" rpy="0 0 0"/>
-                <geometry>
-                    <box size="1 0.6 0.015"/>
-                </geometry>
-            </visual>
-            <inertial>
-                <mass value="1"/>
-                <xacro:box_inertia m="1" x="1" y="0.6" z = "0.015"/>
-            </inertial>
-        </link>
-        <joint name="conveyor_joint" type="fixed">
-            <parent link="base_link"/>
-            <child link="conveyor_belt"/>
-            <origin xyz="0 0 0.25" rpy="0 0 0" />
-        </joint>
-    </xacro:if>
-    <!-- ............................................................................... -->
 </robot>

File: urdf/gz.xacro (robot description, xacro)
@@ -28,23 +28,52 @@
     <!-- ............................. ground truth .................................... -->
     <xacro:if value="${odometry_source == 'world'}">
-    <gazebo>
-        <plugin filename="libgz-sim-odometry-publisher-system"
-            name="gz::sim::systems::OdometryPublisher">
-            <odom_frame>odom</odom_frame>
-            <robot_base_frame>base_footprint</robot_base_frame>
-            <odom_topic>$(arg wheel_odom_topic)</odom_topic>
-            <tf_topic>/tf</tf_topic>
-            <dimensions>2</dimensions>
-            <odom_publish_frequency>10</odom_publish_frequency>
-        </plugin>
-    </gazebo>
+        <gazebo>
+            <plugin filename="libgz-sim-odometry-publisher-system" name="gz::sim::systems::OdometryPublisher">
+                <odom_frame>odom</odom_frame>
+                <robot_base_frame>base_footprint</robot_base_frame>
+                <odom_topic>$(arg wheel_odom_topic)</odom_topic>
+                <tf_topic>/tf</tf_topic>
+                <dimensions>2</dimensions>
+                <odom_publish_frequency>10</odom_publish_frequency>
+            </plugin>
+        </gazebo>
     </xacro:if>
     <!-- ........................... 2D LIDAR config ................................... -->
     <xacro:if value="$(arg two_d_lidar_enabled)">
-        <gazebo reference="two_d_lidar">
-            <sensor name='gpu_lidar' type='gpu_lidar'>
-                <topic>scan</topic>
+        <gazebo reference="L_F_Lidar_Link">
+            <sensor name='lidar_front' type='gpu_lidar'>
+                <topic>lidar_front/scan</topic>
                 <update_rate>${two_d_lidar_update_rate}</update_rate>
-                <gz_frame_id>two_d_lidar</gz_frame_id>
+                <gz_frame_id>L_F_Lidar_Link</gz_frame_id>
+                <lidar>
+                    <scan>
+                        <horizontal>
+                            <samples>${two_d_lidar_sample_size}</samples>
+                            <resolution>1</resolution>
+                            <min_angle>${radians(two_d_lidar_min_angle)}</min_angle>
+                            <max_angle>${radians(two_d_lidar_max_angle)}</max_angle>
+                        </horizontal>
+                    </scan>
+                    <range>
+                        <min>${two_d_lidar_min_range}</min>
+                        <max>${two_d_lidar_max_range}</max>
+                        <resolution>0.01</resolution>
+                    </range>
+                    <noise>
+                        <type>gaussian</type>
+                        <mean>0.0</mean>
+                        <stddev>0.001</stddev>
+                    </noise>
+                </lidar>
+                <always_on>1</always_on>
+                <visualize>true</visualize>
+            </sensor>
+        </gazebo>
+        <!-- ====================== REAR LiDAR ======================== -->
+        <gazebo reference="R_B_Lidar_Link">
+            <sensor name='lidar_rear' type='gpu_lidar'>
+                <topic>lidar_rear/scan</topic>
+                <update_rate>${two_d_lidar_update_rate}</update_rate>
+                <gz_frame_id>R_B_Lidar_Link</gz_frame_id>
                 <lidar>
                     <scan>

File: urdf/ign.xacro (robot description, xacro)
@@ -28,23 +28,22 @@
     <!-- ............................. ground truth .................................... -->
     <xacro:if value="${odometry_source == 'world'}">
-    <gazebo>
-        <plugin filename="libignition-gazebo6-odometry-publisher-system"
-            name="ignition::gazebo::systems::OdometryPublisher">
-            <odom_frame>odom</odom_frame>
-            <robot_base_frame>base_footprint</robot_base_frame>
-            <odom_topic>$(arg wheel_odom_topic)</odom_topic>
-            <tf_topic>/tf</tf_topic>
-            <dimensions>2</dimensions>
-            <odom_publish_frequency>10</odom_publish_frequency>
-        </plugin>
-    </gazebo>
+        <gazebo>
+            <plugin filename="libignition-gazebo6-odometry-publisher-system" name="ignition::gazebo::systems::OdometryPublisher">
+                <odom_frame>odom</odom_frame>
+                <robot_base_frame>base_footprint</robot_base_frame>
+                <odom_topic>$(arg wheel_odom_topic)</odom_topic>
+                <tf_topic>/tf</tf_topic>
+                <dimensions>2</dimensions>
+                <odom_publish_frequency>10</odom_publish_frequency>
+            </plugin>
+        </gazebo>
     </xacro:if>
     <!-- ........................... 2D LIDAR config ................................... -->
     <xacro:if value="$(arg two_d_lidar_enabled)">
-        <gazebo reference="two_d_lidar">
-            <sensor name='gpu_lidar' type='gpu_lidar'>
-                <topic>scan</topic>
+        <gazebo reference="L_F_Lidar_Link">
+            <sensor name='lidar_front' type='gpu_lidar'>
+                <topic>lidar_front/scan</topic>
                 <update_rate>${two_d_lidar_update_rate}</update_rate>
-                <ignition_frame_id>two_d_lidar</ignition_frame_id>
+                <gz_frame_id>L_F_Lidar_Link</gz_frame_id>
                 <lidar>
                     <scan>
@@ -67,5 +66,35 @@
                     </noise>
                 </lidar>
-                <alwaysOn>1</alwaysOn>
+                <always_on>1</always_on>
+                <visualize>true</visualize>
+            </sensor>
+        </gazebo>
+        <!-- ====================== REAR LiDAR ======================== -->
+        <gazebo reference="R_B_Lidar_Link">
+            <sensor name='lidar_rear' type='gpu_lidar'>
+                <topic>lidar_rear/scan</topic>
+                <update_rate>${two_d_lidar_update_rate}</update_rate>
+                <gz_frame_id>R_B_Lidar_Link</gz_frame_id>
+                <lidar>
+                    <scan>
+                        <horizontal>
+                            <samples>${two_d_lidar_sample_size}</samples>
+                            <resolution>1</resolution>
+                            <min_angle>${radians(two_d_lidar_min_angle)}</min_angle>
+                            <max_angle>${radians(two_d_lidar_max_angle)}</max_angle>
+                        </horizontal>
+                    </scan>
+                    <range>
+                        <min>${two_d_lidar_min_range}</min>
+                        <max>${two_d_lidar_max_range}</max>
+                        <resolution>0.01</resolution>
+                    </range>
+                    <noise>
+                        <type>gaussian</type>
+                        <mean>0.0</mean>
+                        <stddev>0.001</stddev>
+                    </noise>
+                </lidar>
+                <always_on>1</always_on>
                 <visualize>true</visualize>
             </sensor>
